File: Hardware/Production/SparkFun u-blox GNSS MAX-M10S-Panel.brd (EAGLE design)
At the start: 203.2 x 137.2 mm, 1414 parts, among them J1 USB-to-Serial, J11 Qwiic RA, J12 PTH, J13 Qwiic RA, J14 USB-to-Serial, J16 Qwiic RA, J17 PTH, J18 Qwiic RA, J19 USB-to-Serial, J2 Qwiic RA, J21 Qwiic RA, J22 PTH, J23 Qwiic RA, J24 USB-to-Serial, J26 Qwiic RA, J27 PTH, J28 Qwiic RA, J29 USB-to-Serial, J3 PTH, J31 Qwiic RA, J32 PTH, J33 Qwiic RA, J34 USB-to-Serial, J36 Qwiic RA, J37 PTH, J38 Qwiic RA, J39 USB-to-Serial, J4 Qwiic RA, J41 Qwiic RA, J42 PTH, J43 Qwiic RA, J44 USB-to-Serial, J46 Qwiic RA, J47 PTH, J48 Qwiic RA, J49 USB-to-Serial, J51 Qwiic RA, J52 PTH, J53 Qwiic RA, J54 USB-to-Serial, J56 Qwiic RA, J57 PTH, J58 Qwiic RA, J59 USB-to-Serial, J6 Qwiic RA, J61 Qwiic RA, J62 PTH, J63 Qwiic RA, J64 USB-to-Serial, J66 Qwiic RA, J67 PTH, J68 Qwiic RA, J69 USB-to-Serial, J7 PTH, J71 Qwiic RA, J72 PTH, J73 Qwiic RA, J74 USB-to-Serial, J76 Qwiic RA, J77 PTH, J78 Qwiic RA, J79 USB-to-Serial, J8 Qwiic RA, J9 USB-to-Serial, U1 MAX-M10S, U10 MAX-M10S, U11 MAX-M10S, U12 MAX-M10S, U13 MAX-M10S, U14 MAX-M10S, U15 MAX-M10S, U16 MAX-M10S, U2 MAX-M10S, U3 MAX-M10S, U4 MAX-M10S, U5 MAX-M10S, U6 MAX-M10S, U7 MAX-M10S, U8 MAX-M10S, U9 MAX-M10S

Commit message: Add panel files
Parts:
- added D33, D36, D39, D42, D45, D48: PESD0402-0402T, SparkFun-DiscreteSemi:0402-TIGHT
- added D34, D37, D40, D43, D46: Yellow, SparkFun-LED:LED-0603
- added D35, D38, D41, D44, D47: 0.5A/40V/420mV, SparkFun-DiscreteSemi:SOD-323
- C1, C10, C12, C14, C16, C18, C20, C22, C24, C26, C28, C30, C32, C4, C6, C8: value 47PF-0402_TIGHT-25V-5%-X7R -> 47pF
- D10, D12, D18, D24, D30, D8: value 0.5A/40V/420mV -> PESD0402-0402T; device SparkFun-DiscreteSemi:SOD-323 -> SparkFun-DiscreteSemi:0402-TIGHT
- D11, D17, D23, D29, D7: value Yellow -> 0.5A/40V/420mV; device SparkFun-LED:LED-0603 -> SparkFun-DiscreteSemi:SOD-323
- D15, D21, D27, D5: value Yellow -> PESD0402-0402T; device SparkFun-LED:LED-0603 -> SparkFun-DiscreteSemi:0402-TIGHT
- D16, D22, D28, D6: value 0.5A/40V/420mV -> Yellow; device SparkFun-DiscreteSemi:SOD-323 -> SparkFun-LED:LED-0603
- E1, E10, E11, E12, E13, E14, E15, E16, E2, E3, E4, E5, E6, E7, E8, E9: value (none) -> ANTENNA-SMA-GROUNDEDEDGE_SMA; device SparkFun-RF:SMA-EDGE-SMD -> SparkFun-RF:SMA-EDGE
- JP1, JP10, JP11, JP12, JP13, JP14, JP15, JP16, JP2, JP3, JP4, JP5, JP6, JP7, JP8, JP9: value (none) -> JUMPER-SMT_3_NO_SILK
- MEAS, MEAS1, MEAS10, MEAS11, MEAS12, MEAS13, MEAS14, MEAS15, MEAS2, MEAS3, MEAS4, MEAS5, MEAS6, MEAS7, MEAS8, MEAS9: value (none) -> JUMPER-COMBO_2_NC_TRACE
- PPS_LED, PPS_LED1, PPS_LED10, PPS_LED11, PPS_LED12, PPS_LED13, PPS_LED14, PPS_LED15, PPS_LED2, PPS_LED3, PPS_LED4, PPS_LED5, PPS_LED6, PPS_LED7, PPS_LED8, PPS_LED9, PWR, PWR1, PWR10, PWR11, PWR12, PWR13, PWR14, PWR15, PWR2, PWR3, PWR4, PWR5, PWR6, PWR7, PWR8, PWR9: value (none) -> JUMPER-SMT_2_NC_TRACE_SILK
- moved D15 128.3 mm to (26.0, 43.5), turned to 90 degrees
- moved D9 119.9 mm to (136.1, 25.4)
- moved D12 98.0 mm to (141.8, 12.5), turned to 90 degrees
- moved D13 88.9 mm to (20.3, 56.4)
- moved D14 88.9 mm to (6.35, 48.8)
- moved D16 81.1 mm to (58.9, 56.4)
- moved D29 75.0 mm to (45.0, 79.8)
- moved D7 70.5 mm to (83.6, 17.8)
- moved D11 69.2 mm to (122.2, 17.8)
- moved D18 68.6 mm to (64.6, 43.5), turned to 90 degrees
- moved D31 64.1 mm to (97.5, 87.4)
- moved D32 64.1 mm to (83.6, 79.8)
- moved D27 58.6 mm to (26.0, 74.5), turned to 90 degrees
- moved D23 49.8 mm to (122.2, 48.8)
- moved D30 47.5 mm to (64.6, 74.5), turned to 90 degrees
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Connections:
- net 3.3V10: now also D32.A; no longer D22.A
- net 3.3V11: now also D35.A; no longer D24.A
- net 3.3V12: now also D38.A; no longer D26.A
- net 3.3V13: now also D41.A; no longer D28.A
- net 3.3V14: now also D44.A; no longer D30.A
- net 3.3V15: now also D47.A; no longer D32.A
- net 3.3V2: now also D7.A; no longer D6.A
- net 3.3V3: now also D11.A; no longer D8.A
- net 3.3V4: now also D14.A; no longer D10.A
- net 3.3V5: now also D17.A; no longer D12.A
- net 3.3V6: now also D20.A; no longer D14.A
- net 3.3V7: now also D23.A; no longer D16.A
- net 3.3V8: now also D26.A; no longer D18.A
- net 3.3V9: now also D29.A; no longer D20.A
- net GND: now also D10.2, E1.GND@2, E1.GND@3
- net GND1: now also D5.2, E2.GND@2, E2.GND@3
- net GND10: now also D31.C, D33.2, E11.GND@2, E11.GND@3; no longer D21.C
- net GND11: now also D34.C, D36.2, E12.GND@2, E12.GND@3; no longer D23.C
- net GND12: now also D37.C, D39.2, E13.GND@2, E13.GND@3; no longer D25.C
- net GND13: now also D40.C, D42.2, E14.GND@2, E14.GND@3; no longer D27.C
- net GND14: now also D43.C, D45.2, E15.GND@2, E15.GND@3; no longer D29.C
- net GND15: now also D46.C, D48.2, E16.GND@2, E16.GND@3; no longer D31.C
- net GND2: now also D6.C, D8.2, E3.GND@2, E3.GND@3; no longer D5.C
- net GND3: now also D12.2, D9.C, E4.GND@2, E4.GND@3; no longer D7.C
- net GND4: now also D13.C, D15.2, E5.GND@2, E5.GND@3; no longer D9.C
- net GND5: now also D16.C, D18.2, E6.GND@2, E6.GND@3; no longer D11.C
- net GND6: now also D19.C, D21.2, E7.GND@2, E7.GND@3; no longer D13.C
- net GND7: now also D22.C, D24.2, E8.GND@2, E8.GND@3; no longer D15.C
- net GND8: now also D25.C, D27.2, E9.GND@2, E9.GND@3; no longer D17.C
- net GND9: now also D28.C, D30.2, E10.GND@2, E10.GND@3; no longer D19.C
- net GPS_RF: now also D10.1
- net GPS_RF1: now also D5.1
- net GPS_RF10: now also D33.1
- net GPS_RF11: now also D36.1
- net GPS_RF12: now also D39.1
- net GPS_RF13: now also D42.1
- net GPS_RF14: now also D45.1
- net GPS_RF15: now also D48.1
- net GPS_RF2: now also D8.1
- net GPS_RF3: now also D12.1
- net GPS_RF4: now also D15.1
- net GPS_RF5: now also D18.1
- net GPS_RF6: now also D21.1
- net GPS_RF7: now also D24.1
- net GPS_RF8: now also D27.1
- net GPS_RF9: now also D30.1
- net N$101: now also D38.C; no longer D26.C
- net N$107: now also D40.A; no longer D27.A
- net N$109: now also D41.C; no longer D28.C
- net N$115: now also D43.A; no longer D29.A
- net N$117: now also D44.C; no longer D30.C
- net N$123: now also D46.A; no longer D31.A
- net N$125: now also D47.C; no longer D32.C
- net N$19: now also D6.A; no longer D5.A
- net N$21: now also D7.C; no longer D6.C
- net N$27: now also D9.A; no longer D7.A
- net N$29: now also D11.C; no longer D8.C
- net N$35: now also D13.A; no longer D9.A
- net N$37: now also D14.C; no longer D10.C
- net N$43: now also D16.A; no longer D11.A
- net N$45: now also D17.C; no longer D12.C
- net N$51: now also D19.A; no longer D13.A
- net N$53: now also D20.C; no longer D14.C
- net N$59: now also D22.A; no longer D15.A
- net N$61: now also D23.C; no longer D16.C
- net N$67: now also D25.A; no longer D17.A
- net N$69: now also D26.C; no longer D18.C
- net N$75: now also D28.A; no longer D19.A
- net N$77: now also D29.C; no longer D20.C
- net N$83: now also D31.A; no longer D21.A
- net N$85: now also D32.C; no longer D22.C
- net N$91: now also D34.A; no longer D23.A
- net N$93: now also D35.C; no longer D24.C
- net N$99: now also D37.A; no longer D25.A
Routing:
- net GPS_RF5: track 9.44 -> 13.5 mm
- net GPS_RF1: track 9.44 -> 13.5 mm
- net GPS_RF9: track 9.44 -> 13.5 mm
- net GPS_RF13: track 9.44 -> 13.5 mm
- net GPS_RF7: track 9.44 -> 13.5 mm
- net GPS_RF4: track 9.44 -> 13.5 mm
- net GPS_RF3: track 9.44 -> 13.5 mm
- net GPS_RF: track 9.44 -> 13.5 mm
- net GPS_RF6: track 9.44 -> 13.5 mm
- net GPS_RF2: track 9.44 -> 13.5 mm
- net GPS_RF8: track 9.44 -> 13.5 mm
- net GPS_RF15: track 9.44 -> 13.5 mm
- net GPS_RF12: track 9.44 -> 13.5 mm
- net GPS_RF11: track 9.44 -> 13.5 mm
- net GPS_RF14: track 9.44 -> 13.5 mm
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Other:
- board size 203.2 x 137.2 mm -> 174 x 137.7 mm
